File: FinalProject/ErgoCompass/ErgoCompass.kicad_sch (KiCad schematic)
At the start: 9 parts, among them J1 Conn_01x02_Socket, J2 FSR406, J3 FSR406, J4 FSR406, U2 XIAO ESP32C3, U3 ADS1115IDGS

Commit message: Update KiCad
Parts:
- added Button1: ~, symbol 113991054:Button
- added D1, D2, D3: NeoPixel_THT, symbol LED:NeoPixel_THT
- added J5: Battery, symbol Connector:Conn_01x02_Socket
- added M1: Stepper_Motor_bipolar, symbol Motor:Stepper_Motor_bipolar
- added U1: XIAO ESP32C3, 113991054:MODULE_113991054, symbol 113991054:XIAO ESP32C3
- added U4: ULN2003A, symbol Transistor_Array:ULN2003A
- J1: value Conn_01x02_Socket -> Battery
Connections:
- new net: D1.1 (DOUT), D2.4 (DIN), U1.6 (D5)
- new net: Button1.2 (S2), D1.2 (GND), D2.2 (GND), D3.2 (GND), U1.13 (GND)
- new net: D1.3 (VDD), D2.3 (VDD), D3.3 (VDD), U1.12 (VCC_3V3)
- new net: D1.4 (DIN), U1.11 (D10)
- new net: D3.4 (DIN), U1.5 (D4)
- new net: Button1.1 (S1), U1.10 (D9)
- new net: U1.1 (D0), U4.1 (I1)
- new net: M1.4, U4.13 (O4)
- new net: M1.3, U4.14 (O3)
- new net: M1.1, U4.15 (O2)
- new net: M1.2 (-), U4.16 (O1)
- new net: U1.2 (D1), U4.2 (I2)
- new net: U1.3 (D2), U4.3 (I3)
- new net: U1.4 (D3), U4.4 (I4)
- new net: J5.1 (Pin_1), U1. (-)
- new net: J5.2 (Pin_2), U1. (-)
Other:
- moved on the sheet: J1, J2, J3, J4, R1, R2, R3, U2, U3
