File: Lab3PCBDesign/Lab3/Lab3.kicad_sch (KiCad schematic)
At the start: 12 parts, among them J1 Conn_01x04_Pin, U1 LM317MBSTT3G, U2 MMC5603NJ

Commit message: Update Lab3
Parts:
- R1: value 50 -> 60
Changed lines of the file:
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@@
 			)
 		)
-		(property "Value" "50"
+		(property "Value" "60"
 			(at 67.31 46.9899 0)
 			(effects
