File: Lab3PCBDesign/Lab3/Lab3.kicad_pcb (KiCad board)
At the start: 2 copper layers, 26.5 x 14.5 mm, 12 parts, among them J1 Conn_01x04_Pin, U1 LM317MBSTT3G, U2 MMC5603NJ

Commit message: Update
Routing:
- net GND: track 5.58 -> 9.95 mm
Changed lines of the file:
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@@
+	(segment
+		(start 124 77.1375)
+		(end 119.8625 77.1375)
+		(width 0.2)
+		(layer "F.Cu")
+		(net 2)
+	)
 	(segment
 		(start 124 77.1375)
@@
 		(width 0.2)
 		(layer "F.Cu")
+		(net 2)
+	)
+	(segment
+		(start 119.8625 77.1375)
+		(end 119.7026 77.2974)
+		(width 0.2)
+		(layer "F.Cu")
