File: FinalProject/Display/Display.kicad_sch (KiCad schematic)
At the start: 7 parts, among them J1 Conn_01x02_Pin, J5 Battery, M1 Stepper_Motor_bipolar

Commit message: Add pdf
Other:
- title: (none) -> Display sch
Changed lines of the file:
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@@
 	(generator_version "9.0")
 	(paper "A4")
+	(title_block
+		(title "Display sch")
+		(date "2026-02-02")
+		(rev "v2")
+	)
 	(junction
 		(at 246.38 73.66)
