File: FinalProject/Sensor/Sensor.kicad_sch (KiCad schematic)
At the start: 9 parts, among them J1 Battery, J2 Conn_01x02_Socket, J3 Conn_01x02_Socket, J4 Conn_01x02_Socket, U3 ADS1115IDGS

Commit message: Add pdf
Other:
- title: (none) -> Sensor sch
Changed lines of the file:
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@@
 	(generator_version "9.0")
 	(paper "A4")
+	(title_block
+		(title "Sensor sch")
+		(date "2026-02-01")
+		(rev "v2")
+	)
 	(junction
 		(at 57.15 104.14)
