File: FinalProject/KiCAD/Display/Display.kicad_sch (KiCad schematic)
At the start: 7 parts, among them J1 Conn_01x02_Pin, J5 Battery, M1 Stepper_Motor_bipolar

Commit message: Organize
Parts:
- removed U2: ~, footprints:XIAO_ESP32, symbol GIX_ESP32:XIAO_ESP32
- added SW1: SW_SPDT, Connector_PinHeader_2.54mm:PinHeader_1x03_P2.54mm_Vertical, symbol Switch:SW_SPDT
- added U1: XIAO ESP32C3, ESP32C3:NEWxiao_esp32c3, symbol NEWxiao_esp32c3 1:XIAO ESP32C3
- J1: footprint Connector_PinHeader_1.00mm:PinHeader_1x02_P1.00mm_Vertical -> Connector_PinHeader_2.54mm:PinHeader_1x02_P2.54mm_Vertical
- J5: footprint Connector_PinSocket_1.00mm:PinSocket_1x02_P1.00mm_Vertical -> Connector_PinSocket_2.54mm:PinSocket_1x02_P2.54mm_Vertical
Connections:
- net +3V3: now also U1.12 (VCC_3V3)
- net +BATT: now also SW1.1 (A), U1.B+ (Batt+); no longer J5.1 (Pin_1)
- net -BATT: now also U1.B- (Batt-)
- net D0: now also U1.1 (D0)
- net D1: now also U1.2 (D1)
- net D10: now also U1.10 (D9)
- net D2: now also U1.3 (D2)
- net D3: now also U1.4 (D3)
- net D6: now also U1.6 (D5)
- net D8: now also U1.8 (D7)
- net D9: now also U1.9 (D8)
- net GND: now also U1.13 (GND)
- new net: J5.1 (Pin_1), SW1.2 (B)
Other:
- moved on the sheet: J5
