File: FinalProject/KiCAD/Sensor/Sensor.kicad_sch (KiCad schematic)
At the start: 9 parts, among them J1 Battery, J2 Conn_01x02_Socket, J3 Conn_01x02_Socket, J4 Conn_01x02_Socket, U3 ADS1115IDGS

Commit message: Code
Parts:
- removed U3: ADS1115IDGS, Package_SO:TSSOP-10_3x3mm_P0.5mm, symbol Analog_ADC:ADS1115IDGS
- added J5: Conn_01x10_Pin, Connector_PinHeader_2.54mm:PinHeader_1x10_P2.54mm_Vertical, symbol Connector:Conn_01x10_Pin
- J1, J2, J3, J4: footprint Connector_PinSocket_1.00mm:PinSocket_1x02_P1.00mm_Vertical -> Connector_PinSocket_2.54mm:PinSocket_1x02_P2.54mm_Vertical
Connections:
- net +3V3: now also J5.1 (Pin_1)
- net GND: now also J5.2 (Pin_2)
- net SCL: now also J5.3 (Pin_3)
- net SDA: now also J5.4 (Pin_4)
- net at J2.1 (Pin_1), R1.2: now also J5.7 (Pin_7)
- net at J3.1 (Pin_1), R2.2: now also J5.8 (Pin_8)
- net at J4.1 (Pin_1), R3.2: now also J5.9 (Pin_9)
Changed lines of the file:
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@@
+	(wire
+		(pts
+			(xy 80.01 99.06) (xy 80.01 148.59)
+		)
+		(stroke
+			(width 0)
+			(type default)
+		)
+	)
 	(wire
 		(pts
@@
 	(wire
 		(pts
+			(xy 87.63 109.22) (xy 87.63 133.35)
+		)
+		(stroke
+			(width 0)
+			(type default)
+		)
+	)
+	(wire
+		(pts
 			(xy 66.04 76.2) (xy 57.15 76.2)
 		)
@@
 	(wire
 		(pts
+			(xy 80.01 148.59) (xy 72.39 148.59)
+		)
+		(stroke
+			(width 0)
+			(type default)
+		)
+	)
+	(wire
+		(pts
 			(xy 44.45 115.57) (xy 48.26 115.57)
 		)
@@
 	(wire
 		(pts
+			(xy 77.47 101.6) (xy 77.47 151.13)
+		)
+		(stroke
+			(width 0)
+			(type default)
+		)
+	)
+	(wire
+		(pts
 			(xy 129.54 96.52) (xy 140.97 96.52)
 		)
@@
 	(wire
 		(pts
-			(xy 87.63 69.85) (xy 87.63 86.36)
+			(xy 87.63 69.85) (xy 87.63 104.14)
 		)
 		(stroke
@@
 	(wire
 		(pts
+			(xy 77.47 151.13) (xy 72.39 151.13)
+		)
+		(stroke
+			(width 0)
+			(type default)
+		)
+	)
+	(wire
+		(pts
 			(xy 161.29 67.31) (xy 161.29 81.28)
 		)
@@
 	(wire
 		(pts
-			(xy 97.79 99.06) (xy 106.68 99.06)
-		)
-		(stroke
-			(width 0)
-			(type default)
-		)
-	)
-	(wire
-		(pts
 			(xy 243.84 95.25) (xy 232.41 95.25)
 		)
@@
 	(wire
 		(pts
+			(xy 82.55 146.05) (xy 72.39 146.05)
+		)
+		(stroke
+			(width 0)
+			(type default)
+		)
+	)
+	(wire
+		(pts
+			(xy 87.63 133.35) (xy 72.39 133.35)
+		)
+		(stroke
+			(width 0)
+			(type default)
+		)
+	)
+	(wire
+		(pts
 			(xy 232.41 97.79) (xy 232.41 113.03)
 		)
@@
 	(wire
 		(pts
+			(xy 97.79 101.6) (xy 97.79 138.43)
+		)
+		(stroke
+			(width 0)
+			(type default)
+		)
+	)
+	(wire
+		(pts
 			(xy 87.63 109.22) (xy 104.14 109.22)
 		)
@@
 	(wire
 		(pts
+			(xy 92.71 130.81) (xy 72.39 130.81)
+		)
+		(stroke
+			(width 0)
+			(type default)
+		)
+	)
+	(wire
+		(pts
+			(xy 92.71 104.14) (xy 92.71 130.81)
+		)
+		(stroke
+			(width 0)
+			(type default)
+		)
+	)
+	(wire
+		(pts
+			(xy 85.09 99.06) (xy 106.68 99.06)
+		)
+		(stroke
+			(width 0)
+			(type default)
+		)
+	)
+	(wire
+		(pts
 			(xy 57.15 97.79) (xy 57.15 96.52)
 		)
@@
 	(wire
 		(pts
+			(xy 85.09 135.89) (xy 72.39 135.89)
+		)
+		(stroke
+			(width 0)
+			(type default)
+		)
+	)
+	(wire
+		(pts
 			(xy 57.15 116.84) (xy 57.15 118.11)
 		)
@@
 	(wire
 		(pts
-			(xy 69.85 99.06) (xy 77.47 99.06)
+			(xy 69.85 99.06) (xy 80.01 99.06)
+		)
+		(stroke
+			(width 0)
+			(type default)
+		)
+	)
+	(wire
+		(pts
+			(xy 82.55 96.52) (xy 82.55 146.05)
 		)
 		(stroke
@@
 	(wire
 		(pts
+			(xy 97.79 138.43) (xy 72.39 138.43)
+		)
+		(stroke
+			(width 0)
+			(type default)
+		)
+	)
+	(wire
+		(pts
 			(xy 48.26 101.6) (xy 48.26 104.14)
 		)
@@
 	(wire
 		(pts
+			(xy 87.63 104.14) (xy 92.71 104.14)
+		)
+		(stroke
+			(width 0)
+			(type default)
+		)
+	)
+	(wire
+		(pts
 			(xy 97.79 101.6) (xy 106.68 101.6)
 		)
@@
 	(wire
 		(pts
-			(xy 69.85 96.52) (xy 77.47 96.52)
+			(xy 69.85 96.52) (xy 82.55 96.52)
 		)
 		(stroke
@@
 		(pts
 			(xy 57.15 90.17) (xy 69.85 90.17)
+		)
+		(stroke
+			(width 0)
+			(type default)
+		)
+	)
+	(wire
+		(pts
+			(xy 85.09 99.06) (xy 85.09 135.89)
 		)
 		(stroke
@@
 			)
 		)
-		(property "Footprint" "Connector_PinSocket_1.00mm:PinSocket_1x02_P1.00mm_Vertical"
+		(property "Footprint" "Connector_PinSocket_2.54mm:PinSocket_1x02_P2.54mm_Vertical"
 			(at 39.37 90.17 0)
 			(effects
@@
 	)
 	(symbol
-		(lib_id "Analog_ADC:ADS1115IDGS")
-		(at 87.63 99.06 0)
-		(unit 1)
-		(exclude_from_sim no)
-		(in_bom yes)
-		(on_board yes)
-		(dnp no)
-		(fields_autoplaced yes)
-		(property "Reference" "U3"
-			(at 89.7733 83.82 0)
-			(effects
-				(font
-					(size 1.27 1.27)
-				)
-				(justify left)
-			)
-		)
-		(property "Value" "ADS1115IDGS"
-			(at 89.7733 86.36 0)
-			(effects
-				(font
-					(size 1.27 1.27)
-				)
-				(justify left)
-			)
-		)
-		(property "Footprint" "Package_SO:TSSOP-10_3x3mm_P0.5mm"
-			(at 87.63 111.76 0)
-			(effects
-				(font
-					(size 1.27 1.27)
-				)
-				(hide yes)
-			)
-		)
-		(property "Datasheet" "http://www.ti.com/lit/ds/symlink/ads1113.pdf"
-			(at 86.36 121.92 0)
-			(effects
-				(font
-					(size 1.27 1.27)
-				)
-				(hide yes)
-			)
-		)
-		(property "Description" "Ultra-Small, Low-Power, I2C-Compatible, 860-SPS, 16-Bit ADCs With Internal Reference, Oscillator, and Programmable Comparator, VSSOP-10"
-			(at 87.63 99.06 0)
-			(effects
-				(font
-					(size 1.27 1.27)
-				)
-				(hide yes)
-			)
-		)
-		(pin "4"
-		)
-		(pin "6"
-		)
-		(pin "5"
-		)
-		(pin "7"
-		)
-		(pin "8"
-		)
-		(pin "3"
-		)
-		(pin "2"
-		)
-		(pin "1"
-		)
-		(pin "9"
-		)
-		(pin "10"
-		)
-		(instances
-			(project "Sensor"
-				(path "/e2176fcb-63e7-4125-a762-1d526a7747a1"
-					(reference "U3")
-					(unit 1)
-				)
-			)
-		)
-	)
-	(symbol
 		(lib_id "power:+3V3")
 		(at 87.63 55.88 0)
@@
 			)
 		)
-		(property "Footprint" "Connector_PinSocket_1.00mm:PinSocket_1x02_P1.00mm_Vertical"
+		(property "Footprint" "Connector_PinSocket_2.54mm:PinSocket_1x02_P2.54mm_Vertical"
 			(at 248.92 95.25 0)
 			(effects
@@
 			)
 		)
-		(property "Footprint" "Connector_PinSocket_1.00mm:PinSocket_1x02_P1.00mm_Vertical"
+		(property "Footprint" "Connector_PinSocket_2.54mm:PinSocket_1x02_P2.54mm_Vertical"
 			(at 39.37 101.6 0)
 			(effects
@@
 				(path "/e2176fcb-63e7-4125-a762-1d526a7747a1"
 					(reference "J3")
+					(unit 1)
+				)
+			)
+		)
+	)
+	(symbol
+		(lib_id "Connector:Conn_01x10_Pin")
+		(at 67.31 140.97 0)
+		(unit 1)
+		(exclude_from_sim no)
+		(in_bom yes)
+		(on_board yes)
+		(dnp no)
+		(fields_autoplaced yes)
+		(property "Reference" "J5"
+			(at 67.945 125.73 0)
+			(effects
+				(font
+					(size 1.27 1.27)
+				)
+			)
+		)
+		(property "Value" "Conn_01x10_Pin"
+			(at 67.945 128.27 0)
+			(effects
+				(font
+					(size 1.27 1.27)
+				)
+			)
+		)
+		(property "Footprint" "Connector_PinHeader_2.54mm:PinHeader_1x10_P2.54mm_Vertical"
+			(at 67.31 140.97 0)
+			(effects
+				(font
+					(size 1.27 1.27)
+				)
+				(hide yes)
+			)
+		)
+		(property "Datasheet" "~"
+			(at 67.31 140.97 0)
+			(effects
+				(font
+					(size 1.27 1.27)
+				)
+				(hide yes)
+			)
+		)
+		(property "Description" "Generic connector, single row, 01x10, script generated"
+			(at 67.31 140.97 0)
+			(effects
+				(font
+					(size 1.27 1.27)
+				)
+				(hide yes)
+			)
+		)
+		(pin "2"
+		)
+		(pin "1"
+		)
+		(pin "5"
+		)
+		(pin "3"
+		)
+		(pin "4"
+		)
+		(pin "7"
+		)
+		(pin "6"
+		)
+		(pin "10"
+		)
+		(pin "9"
+		)
+		(pin "8"
+		)
+		(instances
+			(project ""
+				(path "/e2176fcb-63e7-4125-a762-1d526a7747a1"
+					(reference "J5")
 					(unit 1)
 				)
@@
 			)
 		)
-		(property "Footprint" "Connector_PinSocket_1.00mm:PinSocket_1x02_P1.00mm_Vertical"
+		(property "Footprint" "Connector_PinSocket_2.54mm:PinSocket_1x02_P2.54mm_Vertical"
 			(at 39.37 115.57 0)
 			(effects
